Commit message: Third commit

File: urdf/blueboat.xacro (robot description, xacro)
@@ -45,5 +45,5 @@
       <parent link="${prefix}base_link"/>
       <child link="blueboat/lidar_front"/>
-      <origin xyz="0.0 0.0 -1.2" rpy="3.1416 0 0"/>
+      <origin xyz="0.0 0.0 -1.0" rpy="3.1416 0 0"/>
     </joint>
     <!-- gps Link -->

Commit message: Add real thruster to Blueboat (T200 to M200)

File: urdf/blueboat.xacro (robot description, xacro)
@@ -4,21 +4,26 @@
   <xacro:macro name="blueboat_macro" params="prefix">
     <!-- Base Link -->
-    <link name="${prefix}base_link">
-      <visual>
-        <origin rpy="3.1416 0 -1.5708" xyz="0 0 0" />
-        <geometry>
-          <mesh filename="package://blueboat_stonefish/meshes/blueboat.dae" scale="1 1 1"/>
-        </geometry>
-        <material name="blue">
-          <color rgba="0 0 1 1"/>
-        </material>
-      </visual>
-      <collision>
-        <origin rpy="3.1416 0 -1.5708" xyz="0 0 0" />
-        <geometry>
-          <mesh filename="package://blueboat_stonefish/meshes/blueboat.dae" scale="1 1 1"/>
-        </geometry>
-      </collision>
-    </link>
+  <link name="${prefix}base_link"/>
+  <link name="${prefix}base_link_urdf">
+    <visual>
+      <origin rpy="3.1416 0 -1.5708" xyz="0 0 0"/>
+      <geometry>
+        <mesh filename="package://blueboat_stonefish/meshes/blueboat.dae" scale="1 1 1"/>
+      </geometry>
+      <material name="blue"><color rgba="0 0 1 1"/></material>
+    </visual>
+    <collision>
+      <origin rpy="3.1416 0 -1.5708" xyz="0 0 0"/>
+      <geometry>
+        <mesh filename="package://blueboat_stonefish/meshes/blueboat.dae" scale="1 1 1"/>
+      </geometry>
+    </collision>
+  </link>
+  <joint name="${prefix}base_link_urdf_joint" type="fixed">
+    <parent link="${prefix}base_link"/>
+    <child link="${prefix}base_link_urdf"/>
+    <!-- offset COM -> origen del mesh -->
+    <origin xyz="-0.275 0 -0.23" rpy="0 0 0"/>
+  </joint>
     <!-- Camera link -->
     <link name="blueboat_camera_link">
@@ -29,5 +34,5 @@
     </link>
     <joint name="${prefix}camera_joint" type="fixed">
-      <parent link="${prefix}base_link"/>
+      <parent link="${prefix}base_link_urdf"/>
       <child link="blueboat_camera_link"/>
       <origin xyz="0.45 0.0 0.1" rpy="0 0 0"/>
@@ -43,7 +48,7 @@
     <!-- Joint que une el libox a la base -->
     <joint name="${prefix}lidar_joint" type="fixed">
-      <parent link="${prefix}base_link"/>
+      <parent link="${prefix}base_link_urdf"/>
       <child link="blueboat/lidar_front"/>
-      <origin xyz="0.0 0.0 -1.0" rpy="3.1416 0 0"/>
+      <origin xyz=".39 -0.36 -0.05" rpy="3.1416 0 0"/>
     </joint>
     <!-- gps Link -->
@@ -52,5 +57,5 @@
     <!-- Joint que une el gps a la base -->
     <joint name="${prefix}gps_joint" type="fixed">
-      <parent link="${prefix}base_link"/>
+      <parent link="${prefix}base_link_urdf"/>
       <child link="gps_frame"/>
       <origin xyz=".39 -0.36 -0.05" rpy="3.1416 0 1.57"/>

Commit message: Fixing problems

File: urdf/blueboat.xacro (robot description, xacro)
@@ -27,5 +27,5 @@
   </joint>
     <!-- Camera link -->
-    <link name="blueboat_camera_link">
+    <link name="${prefix}camera_link">
         <visual>
             <geometry><box size="0.05 0.05 0.05"/></geometry>
@@ -35,5 +35,5 @@
     <joint name="${prefix}camera_joint" type="fixed">
       <parent link="${prefix}base_link_urdf"/>
-      <child link="blueboat_camera_link"/>
+      <child link="${prefix}camera_link"/>
       <origin xyz="0.45 0.0 0.1" rpy="0 0 0"/>
     </joint>

Commit message: Fastlio with livox implemented

File: urdf/blueboat.xacro (robot description, xacro)
@@ -1,66 +1,67 @@
 <?xml version="1.0"?>
 <robot xmlns:xacro="http://www.ros.org/wiki/xacro" name="blueboat">
-  <!-- Definir un macro llamado blueboat_macro -->
   <xacro:macro name="blueboat_macro" params="prefix">
-    <!-- Base Link -->
-  <link name="${prefix}base_link"/>
-  <link name="${prefix}base_link_urdf">
-    <visual>
-      <origin rpy="3.1416 0 -1.5708" xyz="0 0 0"/>
-      <geometry>
-        <mesh filename="package://blueboat_stonefish/meshes/blueboat.dae" scale="1 1 1"/>
-      </geometry>
-      <material name="blue"><color rgba="0 0 1 1"/></material>
-    </visual>
-    <collision>
-      <origin rpy="3.1416 0 -1.5708" xyz="0 0 0"/>
-      <geometry>
-        <mesh filename="package://blueboat_stonefish/meshes/blueboat.dae" scale="1 1 1"/>
-      </geometry>
-    </collision>
-  </link>
-  <joint name="${prefix}base_link_urdf_joint" type="fixed">
-    <parent link="${prefix}base_link"/>
-    <child link="${prefix}base_link_urdf"/>
-    <!-- offset COM -> origen del mesh -->
-    <origin xyz="-0.275 0 -0.23" rpy="0 0 0"/>
-  </joint>
-    <!-- Camera link -->
-    <link name="${prefix}camera_link">
-        <visual>
-            <geometry><box size="0.05 0.05 0.05"/></geometry>
-            <material name="blue"/>
-        </visual>
+    <!-- =========================================================
+         1) base_link (ENU) -> lo usa FastLIO como body_frame
+         ========================================================= -->
+    <link name="${prefix}base_link_enu"/>        <!-- ENU -->
+    <link name="${prefix}base_link"/>    <!-- NED -->
+    <joint name="${prefix}enu_to_ned_joint" type="fixed">
+      <parent link="${prefix}base_link_enu"/>
+      <child  link="${prefix}base_link"/>
+      <origin xyz="0 0 0" rpy="3.1416 0 0"/>
+    </joint>
+    <!-- =========================================================
+         3) Mesh solo visual (cuelga del NED físico)
+         ========================================================= -->
+    <link name="${prefix}base_link_urdf">
+      <visual>
+        <origin rpy="3.1416 0 -1.5708" xyz="0 0 0"/>
+        <geometry>
+          <mesh filename="package://blueboat_stonefish/meshes/blueboat.dae" scale="1 1 1"/>
+        </geometry>
+        <material name="blue"><color rgba="0 0 1 1"/></material>
+      </visual>
+      <collision>
+        <origin rpy="3.1416 0 -1.5708" xyz="0 0 0"/>
+        <geometry>
+          <mesh filename="package://blueboat_stonefish/meshes/blueboat.dae" scale="1 1 1"/>
+        </geometry>
+      </collision>
     </link>
+    <joint name="${prefix}base_link_urdf_joint" type="fixed">
+      <parent link="${prefix}base_link"/>
+      <child  link="${prefix}base_link_urdf"/>
+      <origin xyz="-0.275 0 -0.23" rpy="0 0 0"/>
+    </joint>
+    <!-- Cámara (usa offsets de Stonefish) -->
+    <link name="${prefix}camera_link"/>
     <joint name="${prefix}camera_joint" type="fixed">
-      <parent link="${prefix}base_link_urdf"/>
+      <parent link="${prefix}base_link"/>
       <child link="${prefix}camera_link"/>
-      <origin xyz="0.45 0.0 0.1" rpy="0 0 0"/>
+      <origin xyz="0.175 0.0 -0.13" rpy="0.0 0 1.5708"/>
     </joint>
-    <link name="blueboat/lidar_front">
-      <visual>
-        <geometry>
-          <cylinder radius="0.05" length="0.05"/>
-        </geometry>
-        <material name="blue"/>
-      </visual>
-    </link>
-    <!-- Joint que une el libox a la base -->
+    <!-- LiDAR (usa offsets de Stonefish) -->
+    <link name="${prefix}lidar_front"/>
     <joint name="${prefix}lidar_joint" type="fixed">
-      <parent link="${prefix}base_link_urdf"/>
-      <child link="blueboat/lidar_front"/>
-      <origin xyz=".39 -0.36 -0.05" rpy="3.1416 0 0"/>
+      <parent link="${prefix}base_link"/>
+      <child link="${prefix}lidar_front"/>
+      <origin xyz="0.115 -0.36 -0.25" rpy="3.1416 0 0"/>
     </joint>
-    <!-- gps Link -->
-    <link name="gps_frame">
-    </link>
-    <!-- Joint que une el gps a la base -->
+    <!-- GPS (usa offsets de Stonefish) -->
+    <link name="${prefix}gps_frame"/>
     <joint name="${prefix}gps_joint" type="fixed">
-      <parent link="${prefix}base_link_urdf"/>
-      <child link="gps_frame"/>
-      <origin xyz=".39 -0.36 -0.05" rpy="3.1416 0 1.57"/>
+      <parent link="${prefix}base_link"/>
+      <child link="${prefix}gps_frame"/>
+      <origin xyz="-0.35 0.15 +0.35" rpy="0 0 0"/>
+    </joint>
+    <!-- IMU = LiDAR -->
+    <link name="${prefix}imu_link"/>
+    <joint name="${prefix}imu_joint" type="fixed">
+      <parent link="${prefix}base_link"/>
+      <child link="${prefix}imu_link"/>
+      <origin xyz="0.115 -0.36 -0.25" rpy="3.1416 0 0"/>
     </joint>
   </xacro:macro>
-  <!-- LLAMAR A LA MACRO -->
   <xacro:blueboat_macro prefix="blueboat/"/>
 </robot>
